Commit message: Mise à jour avec dépot du projet dééjà existant

File: urdf_models/conserve.urdf (robot description, URDF)
Before this commit: robot obj_model, 1 links, 0 joints
Links:
- link obj_link: mass 1.0 -> 0.425

File: urdf_models/robot_cube.urdf (robot description, URDF)
Before this commit: robot robot_rectangle, 1 links, 0 joints
Links:
- link base: mass None -> 4.0

File: urdf_models/table_eurobot2025.urdf (robot description, URDF)
Before this commit: robot obj_model, 8 links, 7 joints
Links:
- link ramps: geometry collision mesh filename=rampes.obj; visual mesh filename=rampes.obj
- link rendered_table: mass 1.0 -> 1000.0
- link scene: geometry collision box size=0.9 0.45 0.055; visual box size=0 0 0
Joints:
- joint base_to_scene: origin xyz=0 0.78 0.06 rpy=0 0 0 -> xyz=0 0.775 0.05 rpy=0 0 0
